File: OrangeSqueezer.sch (EAGLE design)
At the start: 31 parts, among them IC1 LM4558N, Q1 2N5457, Q2 2N5457

Commit message: Version 1.0 of Pumpkin Pie sent to Oshpark 12/26/15
Parts:
- renumbered +9V1 to +9V, GND1 to G, IN1 to IN, OUT1 to OUT, POT1 to VOL
Changed lines of the file:
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@@
 <?xml version="1.0" encoding="utf-8"?>
 <!DOCTYPE eagle SYSTEM "eagle.dtd">
-<eagle version="7.1.0">
+<eagle version="7.4.0">
 <drawing>
 <settings>
@@
 </classes>
 <parts>
-<part name="+9V1" library="mb_supply" deviceset="+9V(T)" device=""/>
-<part name="GND1" library="mb_supply" deviceset="GND(T)" device=""/>
+<part name="+9V" library="mb_supply" deviceset="+9V(T)" device=""/>
+<part name="G" library="mb_supply" deviceset="GND(T)" device=""/>
 <part name="GND2" library="mb_supply" deviceset="GND" device=""/>
 <part name="GND3" library="mb_supply" deviceset="GND" device=""/>
@@
 <part name="GND5" library="mb_supply" deviceset="GND" device=""/>
 <part name="GND6" library="mb_supply" deviceset="GND" device=""/>
-<part name="IN1" library="mb_supply" deviceset="IN(T)" device=""/>
-<part name="OUT1" library="mb_supply" deviceset="OUT(T)" device=""/>
+<part name="IN" library="mb_supply" deviceset="IN(T)" device=""/>
+<part name="OUT" library="mb_supply" deviceset="OUT(T)" device=""/>
 <part name="R1" library="mb_resistors" deviceset="6MM" device=".3" value="1M5"/>
 <part name="R2" library="mb_resistors" deviceset="6MM" device=".3" value="82k"/>
@@
 <part name="Q2" library="mb_trans" deviceset="2N5457" device=""/>
 <part name="IC1" library="mb_ics" deviceset="*4558" device="N" technology="LM"/>
-<part name="POT1" library="mb_pots" deviceset="POT" device="16MM_PCB_PADS" value="A10k"/>
+<part name="VOL" library="mb_pots" deviceset="POT" device="16MM_PCB_PADS" value="A10k"/>
 <part name="POT2" library="mb_pots" deviceset="POT" device="TRIM" value="10k"/>
 <part name="D1" library="mb_diodes" deviceset="1N400X" device=".3" value="1N34A"/>
@@
 </plain>
 <instances>
-<instance part="+9V1" gate="+9V" x="-7.62" y="86.36" rot="R90"/>
-<instance part="GND1" gate="GND" x="-2.54" y="50.8"/>
+<instance part="+9V" gate="+9V" x="-7.62" y="86.36" rot="R90"/>
+<instance part="G" gate="GND" x="-2.54" y="50.8"/>
 <instance part="GND2" gate="GND" x="50.8" y="15.24"/>
 <instance part="GND3" gate="GND" x="38.1" y="15.24"/>
@@
 <instance part="GND5" gate="GND" x="27.94" y="15.24"/>
 <instance part="GND6" gate="GND" x="68.58" y="15.24"/>
-<instance part="IN1" gate="G$1" x="-7.62" y="68.58"/>
-<instance part="OUT1" gate="G$1" x="116.84" y="58.42"/>
+<instance part="IN" gate="G$1" x="-7.62" y="68.58"/>
+<instance part="OUT" gate="G$1" x="116.84" y="58.42"/>
 <instance part="R1" gate="G$1" x="-2.54" y="60.96" rot="R90"/>
 <instance part="R2" gate="G$1" x="15.24" y="68.58"/>
@@
 <instance part="Q1" gate="G$1" x="10.16" y="48.26" rot="R180"/>
 <instance part="Q2" gate="G$1" x="27.94" y="55.88" rot="R180"/>
-<instance part="POT1" gate="G$1" x="106.68" y="58.42"/>
+<instance part="VOL" gate="G$1" x="106.68" y="58.42"/>
 <instance part="POT2" gate="G$1" x="40.64" y="27.94"/>
 <instance part="D1" gate="1" x="93.98" y="50.8" rot="R270"/>
@@
 <net name="IN" class="0">
 <segment>
-<pinref part="IN1" gate="G$1" pin="IN"/>
+<pinref part="IN" gate="G$1" pin="IN"/>
 <pinref part="C1" gate="G$1" pin="2"/>
 <wire x1="-5.08" y1="68.58" x2="-2.54" y2="68.58" width="0.1524" layer="91"/>
@@
 </segment>
 <segment>
-<pinref part="POT1" gate="G$1" pin="1"/>
+<pinref part="VOL" gate="G$1" pin="1"/>
 <pinref part="GND9" gate="GND" pin="GND"/>
 <wire x1="104.14" y1="50.8" x2="104.14" y2="17.78" width="0.1524" layer="91"/>
 </segment>
 <segment>
-<pinref part="GND1" gate="GND" pin="GND"/>
+<pinref part="G" gate="GND" pin="GND"/>
 <pinref part="R1" gate="G$1" pin="1"/>
 <wire x1="-2.54" y1="53.34" x2="-2.54" y2="55.88" width="0.1524" layer="91"/>
@@
 <wire x1="83.82" y1="66.04" x2="88.9" y2="66.04" width="0.1524" layer="91"/>
 <wire x1="88.9" y1="66.04" x2="88.9" y2="58.42" width="0.1524" layer="91"/>
-<pinref part="POT1" gate="G$1" pin="3"/>
+<pinref part="VOL" gate="G$1" pin="3"/>
 <wire x1="88.9" y1="66.04" x2="104.14" y2="66.04" width="0.1524" layer="91"/>
 <junction x="88.9" y="66.04"/>
@@
 <segment>
 <pinref part="R14" gate="G$1" pin="1"/>
-<pinref part="+9V1" gate="+9V" pin="+9V"/>
+<pinref part="+9V" gate="+9V" pin="+9V"/>
 <wire x1="-2.54" y1="91.44" x2="-2.54" y2="86.36" width="0.1524" layer="91"/>
 <wire x1="-2.54" y1="86.36" x2="-5.08" y2="86.36" width="0.1524" layer="91"/>
@@
 <net name="OUT" class="0">
 <segment>
-<pinref part="POT1" gate="G$1" pin="2"/>
-<pinref part="OUT1" gate="G$1" pin="OUT"/>
+<pinref part="VOL" gate="G$1" pin="2"/>
+<pinref part="OUT" gate="G$1" pin="OUT"/>
 <wire x1="109.22" y1="58.42" x2="114.3" y2="58.42" width="0.1524" layer="91"/>
 </segment>

Commit message: First commit for The Thing tremolo
Parts:
- removed +9V: +9V(T), mb_supply:+9V(T)
- removed G: GND(T), mb_supply:GND(T)
- removed IN: IN(T), mb_supply:IN(T)
- removed LED: LED, mb_supply:PAD
- removed OUT: OUT(T), mb_supply:OUT(T)
- added Q3, Q4: 2N5457, xc_library:2N5457
- added U$1: BOARDLINK, xc_library:BOARDLINK
- C1, C4: value 0.047uF -> 47nF
- C2: value 0.0022uF -> 2n2
- Q1, Q2: value 2N5457 -> MMBF5457; device mb_trans:2N5457 -> xc_library:MMBF5457
Connections:
- removed net IN: C1.2, IN.IN, R1.2
- removed net OUT: OUT.OUT, VOL.2
- new net N$10: U$1.OUT, VOL.2
- new net N$20: C1.2, R1.2, U$1.IN
- net +9V: now also Q3.S, U$1.+9V; no longer +9V.+9V
- net GND: now also U$1.G; no longer G.GND
- net N$16: now also U$1.LED; no longer LED.PAD
- net N$2: now also Q3.D
- net N$3: now also Q3.G, Q4.D
- net N$5: now also Q4.S
- net N$7: now also Q4.G
Other:
- moved on the sheet: D2, R14
